Commit message: Add robot description.

File: ros_ws/src/snd_description/urdf/macros.xacro (robot description, xacro)
@@ -1,4 +1,5 @@
 <?xml version="1.0"?>
 <robot xmlns:xacro="http://www.ros.org/wiki/xacro" name="macros">
+    <xacro:property name="PI" value="3.141592654"/>
     <xacro:macro name="cylinder_inertia" params="m r h">
         <inertia

File: ros_ws/src/snd_description/urdf/robot_base.urdf.xacro (robot description, xacro)
@@ -8,10 +8,10 @@
     <xacro:property name="encoders_wheel_width" value="0.03"/>
     <xacro:property name="encoders_wheel_separation" value="0.995"/>
-    <xacro:property name="body_length" value="0.106"/>
-    <xacro:property name="body_width" value="0.1415"/>
-    <xacro:property name="body_height" value="0.08878"/>
+    <xacro:property name="body_length" value="0.23"/>
+    <xacro:property name="body_width" value="0.28"/>
+    <xacro:property name="body_height" value="0.32"/>
     <!-- distance between floor and base of robot body -->
     <xacro:property name="robot_clearance" value="0.010"/>
-    <xacro:property name="robot_weight" value="1.0"/>
+    <xacro:property name="robot_weight" value="4.0"/>
     <xacro:property name="caster_radius" value="0.005"/>
     <material name="dark_grey">
@@ -27,9 +27,4 @@
         <color rgba="0.0 0.0 0.7 1.0"/>
     </material>
-    <!--gazebo>
-        <plugin name="gazebo_ros_control" filename="libgazebo_ros_control.so">
-            <robotNamespace>/</robotNamespace>
-        </plugin>
-    </gazebo-->
     <xacro:macro name="robot_body">
         <link name="base_link"></link>
@@ -43,12 +38,12 @@
             </visual-->
             <visual>
-                <origin xyz="0 0 -0.01" rpy="0 0 -${pi/2}"/>
+                <origin xyz="0 0 ${-0.01 - body_height/2}" rpy="0 0 ${pi/2}"/>
                 <geometry>
-                    <mesh filename="package://snd_description/meshes/robot_base_simple.stl" scale="0.001 0.001 0.001"/>
+                    <mesh filename="package://snd_description/meshes/snd_robot_base.dae" scale="1 1 1"/>
                 </geometry>
                 <material name="dark_grey"/>
             </visual>
             <collision>
-                <orign xyz="0 0 0" rpy="0 0 0"/>
+                <orign xyz="0.0 0 0" rpy="0 0 0"/>
                 <geometry>
                     <box size="${body_length} ${body_width} ${body_height}"/>
@@ -56,5 +51,5 @@
             </collision>
             <inertial>
-                <orign xyz="0 0 0" rpy="0 0 0"/>
+                <orign xyz="0.0 0 0" rpy="0 0 0"/>
                 <mass value="${robot_weight}"/>
                 <xacro:box_inertia m="${robot_weight}" x="${body_length}" y="${body_width}" z="${body_height}"/>
@@ -64,5 +59,5 @@
             <parent link="base_link"/>
             <child link="robot_body"/>
-            <origin xyz="0 0 ${robot_clearance}" rpy="0 0 0"/>
+            <origin xyz="0 0 ${body_height/2 + robot_clearance}" rpy="0 0 0"/>
         </joint>
         <xacro:macro name="wheel" params="prefix ypos dir">
@@ -90,6 +85,6 @@
                 <inertial>
                     <origin xyz="0 0 0" rpy="0 ${pi/2} 0"/>
-                    <mass value="0.05"/>
-                    <xacro:cylinder_inertia m="0.2" r="${motor_wheel_radius}" h="${motor_wheel_width}"/>
+                    <mass value="0.1"/>
+                    <xacro:cylinder_inertia m="0.1" r="${motor_wheel_radius}" h="${motor_wheel_width}"/>
                 </inertial>
             </link>
@@ -103,5 +98,5 @@
                 <type>transmission_interface/SimpleTransmission</type>
                 <joint name="${prefix}_wheel_joint">
-                    <hardwareInterface>VelocityJointInterface</hardwareInterface>
+                    <hardwareInterface>hardware_interface/VelocityJointInterface</hardwareInterface>
                 </joint>
                 <actuator name="${prefix}_wheel_actuator">
@@ -116,5 +111,5 @@
         <xacro:wheel prefix="left"  ypos="${motor_wheel_separation / 2.0}" dir="1"/>
         <xacro:wheel prefix="right" ypos="-${motor_wheel_separation / 2.0}" dir="-1"/>
-        <!--xacro:macro name="caster" params="prefix position">
+        <xacro:macro name="caster" params="prefix position">
             <link name="${prefix}_caster">
                 <visual>
@@ -138,5 +133,5 @@
             </link>
             <joint name="base_to_${prefix}_caster" type="fixed">
-                <parent link="robot_up_plate"/>
+                <parent link="base_link"/>
                 <child link="${prefix}_caster"/>
                 <origin xyz="${position}" rpy="0 0 0"/>
@@ -147,6 +142,6 @@
             </gazebo>
         </xacro:macro>
-        <xacro:caster prefix="left" position="${body_length / 2.0 - 0.05} 0.16 -${body_height + caster_radius}"/>
-        <xacro:caster prefix="right" position="${body_length / 2.0 - 0.05} -0.16 -${body_height + caster_radius}"/-->
+        <xacro:caster prefix="front" position="0.1016 0 ${caster_radius + 0.001}"/>
+        <xacro:caster prefix="rear" position="-0.065 0 ${caster_radius + 0.003}"/>
         <gazebo>
             <plugin name="differential_drive_controller" filename="libgazebo_ros_diff_drive.so">
@@ -163,5 +158,7 @@
                 <robotBaseFrame>base_link</robotBaseFrame>
                 <legacyMode>false</legacyMode>
+                <publishTF>true</publishTF>
                 <publishWheelTF>true</publishWheelTF>
+                <publishWheelJointState>true</publishWheelJointState>
             </plugin>
         </gazebo>

File: ros_ws/src/snd_description/urdf/snd_robot.urdf.xacro (robot description, xacro)
@@ -1,5 +1,53 @@
 <?xml version="1.0"?>
 <robot xmlns:xacro="http://www.ros.org/wiki/xacro" name="snd_robot">
+    <xacro:include filename="$(find snd_description)/urdf/macros.xacro"/>
     <xacro:include filename="$(find snd_description)/urdf/robot_base.urdf.xacro"/>
     <xacro:robot_body/>
+    <!--gazebo>
+        <plugin name="gazebo_ros_control" filename="libgazebo_ros_control.so">
+            <robotNamespace>/snd_robot</robotNamespace>
+        </plugin>
+    </gazebo-->
+    <!-- Rplidar -->
+    <xacro:include filename="$(find snd_description)/urdf/sensors/rplidara2.urdf.xacro"/>
+    <xacro:sensor_rplidara2 parent="base_link">
+        <origin xyz="0.085 -0.07 0.03" rpy="0 0 1.570796327"/>
+    </xacro:sensor_rplidara2>
+    <!-- Module arm -->
+    <link name="arm">
+        <visual>
+            <origin xyz="-0.045 0 -0.006" rpy="0 0 ${pi/2}"/>
+            <geometry>
+                <mesh filename="package://snd_description/meshes/arm.stl" scale="1 1 1"/>
+            </geometry>
+            <material name="blue"/>
+        </visual>
+        <collision>
+            <origin xyz="0 -0.05 0" rpy=" ${pi/2} 0 0"/>
+            <geometry>
+                <cylinder length="0.130" radius="0.0275"/>
+            </geometry>
+        </collision>
+        <inertial>
+            <origin xyz="0 -0.05 0" rpy="${pi/2} 0 0"/>
+            <mass value="0.005"/>
+            <xacro:cylinder_inertia m="0.005" r="0.0275" h="0.130"/>
+        </inertial>
+    </link>
+    <!--joint name="arm_servo_joint" type="continuous"-->
+    <joint name="arm_servo_joint" type="fixed">
+        <parent link="base_link"/>
+        <child link="arm"/>
+        <origin xyz="0.025 0.15 0.05" rpy="0 0 ${pi/2}"/>
+        <axis xyz="1 0 0"/>
+    </joint>
+    <!--transmission name="arm_transmission">
+        <type>transmission_interface/SimpleTransmission</type>
+        <joint name="arm_servo_joint">
+            <hardwareInterface>hardware_interface/EffortJointInterface</hardwareInterface>
+        </joint>
+        <actuator name="arm_actuator">
+            <mechanicalReduction>1</mechanicalReduction>
+        </actuator>
+    </transmission-->
 </robot>
