Commit message: Add Gazebo plugin and associated actions servers for Polar Control Loop
- Add a Gazebo plugin simulating the real robot, sending wheels speeds and reading encoders counts
- Add actions using about the same control loop as in the microcontroller
- Add a tester node that call action clients from the command line
- Add a node to move along a square

Note, for now, the command is not a PWM (-10000 10000) but wheels speeds in rad/s so the PID has different tunings.

File: ros_ws/src/snd_description/urdf/simple_robot_base.urdf.xacro (robot description, xacro)
@@ -5,7 +5,4 @@
     <xacro:property name="motor_wheel_width" value="0.011"/>
     <xacro:property name="motor_wheel_separation" value="0.23"/>
-    <xacro:property name="encoders_wheel_radius" value="0.026"/>
-    <xacro:property name="encoders_wheel_width" value="0.03"/>
-    <xacro:property name="encoders_wheel_separation" value="0.995"/>
     <xacro:property name="body_length" value="0.20"/>
     <xacro:property name="body_width" value="0.20"/>
@@ -130,23 +127,4 @@
         <xacro:caster prefix="front" position="0.08 0 ${caster_radius + 0.001}"/>
         <xacro:caster prefix="rear" position="-0.08 0 ${caster_radius + 0.001}"/>
-        <gazebo>
-            <plugin name="differential_drive_controller" filename="libgazebo_ros_diff_drive.so">
-                <alwaysOn>true</alwaysOn>
-                <updateRate>20</updateRate>
-                <leftJoint>left_wheel_joint</leftJoint>
-                <rightJoint>right_wheel_joint</rightJoint>
-                <wheelSeparation>${motor_wheel_separation}</wheelSeparation>
-                <wheelDiameter>${2.0 * motor_wheel_radius}</wheelDiameter>
-                <torque>20</torque>
-                <commandTopic>cmd_vel</commandTopic>
-                <odometryTopic>odom</odometryTopic>
-                <odometryFrame>odom</odometryFrame>
-                <robotBaseFrame>base_link</robotBaseFrame>
-                <legacyMode>false</legacyMode>
-                <publishTf>true</publishTf>
-                <publishWheelTF>true</publishWheelTF>
-                <publishWheelJointState>true</publishWheelJointState>
-            </plugin>
-        </gazebo>
     </xacro:macro>
 </robot>

File: ros_ws/src/snd_description/urdf/simple_robot_lowlevel.urdf.xacro (robot description, xacro)
@@ -4,5 +4,5 @@
     <xacro:include filename="$(find snd_description)/urdf/simple_robot_base.urdf.xacro"/>
     <xacro:robot_body/>
-    <xacro:include filename="$(find snd_description)/urdf/simple_robot_gazebo.xacro"/>
+    <xacro:include filename="$(find snd_description)/urdf/simple_robot_lowlevel_gazebo.xacro"/>
     <!-- Rplidar -->
     <xacro:include filename="$(find snd_description)/urdf/sensors/rplidara2.urdf.xacro"/>
