Commit message: Update simple robot description

File: ros_ws/src/snd_description/urdf/sensors/rplidara2.urdf.xacro (robot description, xacro)
@@ -48,5 +48,5 @@
                     <range>
                         <min>0.15</min>
-                        <max>8</max>
+                        <max>3</max>
                         <resolution>0.01</resolution>
                     </range>

File: ros_ws/src/snd_description/urdf/simple_robot.urdf.xacro (robot description, xacro)
@@ -8,5 +8,5 @@
     <xacro:include filename="$(find snd_description)/urdf/sensors/rplidara2.urdf.xacro"/>
     <xacro:sensor_rplidara2 parent="base_link">
-        <origin xyz="0.0 0.0 0.05" rpy="0 0 1.570796327"/>
+        <origin xyz="0.0 0.0 ${body_height + 0.05}" rpy="0 0 1.570796327"/>
     </xacro:sensor_rplidara2>
 </robot>

File: ros_ws/src/snd_description/urdf/simple_robot_base.urdf.xacro (robot description, xacro)
@@ -5,11 +5,13 @@
     <xacro:property name="motor_wheel_width" value="0.011"/>
     <xacro:property name="motor_wheel_separation" value="0.23"/>
-    <xacro:property name="body_length" value="0.20"/>
-    <xacro:property name="body_width" value="0.20"/>
-    <xacro:property name="body_height" value="0.25"/>
+    <xacro:property name="body_length" value="0.23"/>
+    <xacro:property name="body_width" value="0.265"/>
+    <xacro:property name="body_height" value="0.32"/>
     <!-- distance between floor and base of robot body -->
     <xacro:property name="robot_clearance" value="0.010"/>
     <xacro:property name="robot_weight" value="4.0"/>
     <xacro:property name="caster_radius" value="0.005"/>
+    <xacro:property name="beacon_mast_height" value="0.095"/>
+    <xacro:property name="beacon_mast_radius" value="0.050"/>
     <material name="dark_grey">
         <color rgba="0.2 0.2 0.2 1"/>
@@ -50,4 +52,30 @@
             <child link="robot_body"/>
             <origin xyz="0 0 ${body_height/2 + robot_clearance}" rpy="0 0 0"/>
+        </joint>
+        <link name="beacon_mast">
+            <visual>
+                <orign xyz="0 0 0" rpy="0 0 0"/>
+                <geometry>
+                    <cylinder length="${beacon_mast_height}" radius="${beacon_mast_radius}"/>
+                </geometry>
+                <material name="blue"/>
+            </visual>
+            <collision>
+                <orign xyz="0 0 0" rpy="0 0 0"/>
+                <geometry>
+                    <cylinder length="${beacon_mast_height}" radius="${beacon_mast_radius}"/>
+                </geometry>
+                <material name="blue"/>
+            </collision>
+            <inertial>
+                <orign xyz="0 0 0" rpy="0 0 0"/>
+                <mass value="0.01"/>
+                <xacro:cylinder_inertia m="0.1" r="${motor_wheel_radius}" h="${motor_wheel_width}"/>
+            </inertial>
+        </link>
+        <joint name="mast_to_body" type="fixed">
+            <parent link="base_link"/>
+            <child link="beacon_mast"/>
+            <origin xyz="0 0 ${body_height + robot_clearance + beacon_mast_height / 2}" rpy="0 0 0"/>
         </joint>
         <xacro:macro name="wheel" params="prefix ypos dir">

File: ros_ws/src/snd_description/urdf/simple_robot_gazebo.xacro (robot description, xacro)
@@ -8,4 +8,6 @@
                 <rightJoint>right_wheel_joint</rightJoint>
                 <wheelSeparation>${motor_wheel_separation}</wheelSeparation>
+                <wheelAcceleration>0</wheelAcceleration>
+                <wheelTorque>5</wheelTorque>
                 <wheelDiameter>${2.0 * motor_wheel_radius}</wheelDiameter>
                 <torque>20</torque>
@@ -13,4 +15,5 @@
                 <odometryTopic>odom</odometryTopic>
                 <odometryFrame>odom</odometryFrame>
+                <odometrySource>1</odometrySource>
                 <robotBaseFrame>base_link</robotBaseFrame>
                 <legacyMode>false</legacyMode>
@@ -18,4 +21,5 @@
                 <publishWheelTF>true</publishWheelTF>
                 <publishWheelJointState>true</publishWheelJointState>
+                <rosDebugLevel>0</rosDebugLevel>
             </plugin>
         </gazebo>
